File: light sensor basic.brd (EAGLE design)
At the start: 83.2 x 57.8 mm, 1 part

Commit message: eagle assignment 2
Parts:
- added C1: 0.1uF, rcl:C1206
- added J1: UJ2-MIBH-G-SMT-TR, UJ2-MIBH-G-SMT-TR:CUI_UJ2-MIBH-G-SMT-TR
- added LED1: 500, led:SML0805
- added R1: 82, rcl:R1206
- added R2: TC33X-2-203E, TC33X-2-203E:TRIM_TC33X-2-203E
- added R3, TP3: 150, rcl:R0805
- added T1: (no value), transistor:SOT23-EBC
- added TP1, TP2, TP4: (no value), rcl:R1206
- added U1: VCNT2020, VCNT2020:XDCR_VCNT2020
Connections:
- new net GND: C1.1, J1.5, J1.S1, J1.S2, J1.S3, J1.S4, R2.3, T1.E, TP4.1, TP4.2, U1.4
- new net N$1: R1.1, U1.3
- new net N$2: R2.2, T1.B, TP2.1, TP2.2
- new net N$3: LED1.C, T1.C
- new net N$4: R2.1, TP1.1, TP1.2, U1.1
- new net N$5: LED1.A, R3.1
- new net VCC: C1.2, J1.1, R1.2, R3.2, TP3.1, TP3.2, U1.2
Routing:
- net VCC: track 0.00 -> 48.2 mm
- net N$4: track 0.00 -> 42.3 mm
- net GND: track 0.00 -> 12.3 mm
- net N$2: track 0.00 -> 8.14 mm
- net N$3: track 0.00 -> 6.11 mm
- net N$1: track 0.00 -> 5.82 mm
- net N$5: track 0.00 -> 5.62 mm
- added copper zone on layer 1, net GND
Other:
- board text added: "C1"
- board text added: "J1"
- board text added: "K"
- board text added: "LED1"
- board text added: "R1"
- board text added: "R2"
- board text added: "R3"
- board text added: "T1"
- board text added: "TP1"
- board text added: "TP2"
- board text added: "TP3"
- board text added: "U1"
